Commit message: updated urdf and navigation

File: install/kinclong_nav/share/kinclong_nav/urdf/mogi_bot.urdf (robot description, URDF)
Before this commit: robot mogi_bot, 5 links, 4 joints
Links:
- link base_link: geometry collision cylinder length=0.1 radius=0.2; visual mesh filename=package://kinclong_nav/meshes/body.stl
- link left_wheel: mass 5.0 -> 0.3; geometry collision cylinder length=0.025 radius=0.0325; visual mesh filename=package://kinclong_nav/meshes/roda.stl
- link right_wheel: mass 5.0 -> 0.3; geometry collision cylinder length=0.025 radius=0.0325; visual mesh filename=package://kinclong_nav/meshes/roda.stl
- link scan_link: geometry collision box size=.1 .1 .1; visual mesh filename=package://kinclong_nav/meshes/lidar.stl
Joints:
- joint base_footprint_joint: origin xyz=0 0 0 rpy=0 0 0 -> xyz=0 0 0 rpy=0 0 -1.5707
- joint left_wheel_joint: axis 0 1 0 -> -1 0 0; limit effort=100 velocity=10 -> effort=100 velocity=10.0; origin xyz=0 0.15 0 rpy=0 0 0 -> xyz=-0.142 0 0.03 rpy=0 0 0 
- joint right_wheel_joint: axis 0 1 0 -> -1 0 0; limit effort=100 velocity=10 -> effort=100 velocity=10.0; origin xyz=0 -0.15 0 rpy=0 0 0 -> xyz=0.142 0 0.03 rpy=0 0 0
- joint scan_joint: origin xyz=0.0 0 0.15 rpy=0 0 0 -> xyz=0 0.09 0.12 rpy=0 0 0
